File: MCU_Power.kicad_sch (KiCad schematic)
At the start: 2 parts

Commit message: first draft schematic?
Parts:
- gave numbers to parts that had none: 2
Changed lines of the file:
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@@
   (symbol (lib_id "Reference_Voltage:ADR4530") (at 203.2 96.52 0) (unit 1)
     (in_bom yes) (on_board yes)
-    (property "Reference" "U?" (id 0) (at 203.2 90.17 0))
+    (property "Reference" "U44" (id 0) (at 203.2 90.17 0))
     (property "Value" "ADR4530" (id 1) (at 205.74 102.87 0))
     (property "Footprint" "Package_SO:SOIC-8_3.9x4.9mm_P1.27mm" (id 2) (at 205.74 104.14 0)
@@
   (symbol (lib_id "power:+3V3") (at 226.06 86.36 0) (unit 1)
     (in_bom yes) (on_board yes)
-    (property "Reference" "#PWR?" (id 0) (at 226.06 90.17 0)
+    (property "Reference" "#PWR0147" (id 0) (at 226.06 90.17 0)
       (effects (font (size 1.27 1.27)) hide)
     )
@@
   (symbol (lib_id "power:GND") (at 226.06 106.68 0) (unit 1)
     (in_bom yes) (on_board yes)
-    (property "Reference" "#PWR?" (id 0) (at 226.06 113.03 0)
+    (property "Reference" "#PWR0148" (id 0) (at 226.06 113.03 0)
       (effects (font (size 1.27 1.27)) hide)
     )
@@
   (symbol (lib_id "power:GND") (at 200.66 106.68 0) (unit 1)
     (in_bom yes) (on_board yes)
-    (property "Reference" "#PWR?" (id 0) (at 200.66 113.03 0)
+    (property "Reference" "#PWR0146" (id 0) (at 200.66 113.03 0)
       (effects (font (size 1.27 1.27)) hide)
     )
@@
   (symbol (lib_id "STM32G473QET6:STM32G473QET6") (at 241.3 96.52 0) (mirror y) (unit 8)
     (in_bom yes) (on_board yes)
-    (property "Reference" "U?" (id 0) (at 248.92 86.36 0)
+    (property "Reference" "U3" (id 0) (at 248.92 86.36 0)
       (effects (font (size 1.27 1.27)) (justify left bottom))
     )
@@
   (symbol (lib_id "power:+3V3") (at 200.66 86.36 0) (unit 1)
     (in_bom yes) (on_board yes)
-    (property "Reference" "#PWR?" (id 0) (at 200.66 90.17 0)
-      (effects (font (size 1.27 1.27)) hide)
-    )
+    (property "Reference" "#PWR0145" (id 0) (at 200.66 90.17 0)
+      (effects (font (size 1.27 1.27)) hide)
+    )
