File: TimerBuffers.kicad_sch (KiCad schematic)
At the start: 4 parts

Commit message: first draft schematic?
Parts:
- added C67, C68, C69, C70, C71, C72, C73, C74, C75, C76, C77, C78: C_Small, Capacitor_SMD:C_0603_1608Metric, symbol Device:C_Small
- added U40, U41: ADuM120N, Package_SO:SOIC-8_3.9x4.9mm_P1.27mm, symbol Isolator:ADuM120N
- gave numbers to parts that had none: 4
Connections:
- net +3V3: now also C67.1, C68.1, C69.1, C70.1, C71.1, C72.1, U40.1 (VDD1), U41.1 (VDD1)
- net +5V: now also C73.1, C74.1, C75.1, C76.1, C77.1, C78.1, U40.8 (VDD2), U41.8 (VDD2)
- net GND: now also C67.2, C68.2, C69.2, C70.2, C71.2, C72.2, U40.4 (GND1), U41.4 (GND1)
- net GND1: now also C73.2, C74.2, C75.2, C76.2, C77.2, C78.2, U40.5 (GND2), U41.5 (GND2)
- net PWM_O_1: now also U40.7 (VOA)
- net PWM_O_2: now also U40.6 (VOB)
- net PWM_O_3: now also U41.7 (VOA)
- net PWM_O_4: now also U41.6 (VOB)
- new net PWM_I_5: U40.2 (VIA)
- new net PWM_I_6: U40.3 (VIB)
- new net PWM_I_7: U41.2 (VIA)
- new net PWM_I_8: U41.3 (VIB)
Other:
- moved on the sheet: U39, U42, U43, U5
