File: comms.kicad_sch (KiCad schematic)
At the start: 4 parts, among them U35 ADuM121N, U36 ISO1050DUB, U37 ADuM1250, U38 ADuM3153

Commit message: first draft schematic?
Parts:
- added C59, C60, C61, C62, C63, C64, C65, C66: C_Small, Capacitor_SMD:C_0603_1608Metric, symbol Device:C_Small
Connections:
- net +3V3: now reaches U37.1 (VDD1)
- net +3V3: now also U35.1 (VDD1), U36.1 (VCC1), U38.1 (V_{DD1}), C59.1, C60.1, C61.1, C62.1
- net I2C_SDA: now reaches U37.2 (SDA1)
- net I2C_SCL: now reaches U37.3 (SCL1)
- net GND: now reaches U37.4 (GND1)
- net GND: now also U35.4 (GND1), U36.4 (GND1), U38.10 (GND_{1}), U38.2 (GND_{1}), C59.2, C60.2, C61.2, C62.2
- net GND1: now reaches U37.5 (GND2)
- net GND1: now also U35.5 (GND2), U36.5 (GND2), U38.11 (GND_{2}), U38.19 (GND_{2}), C63.2, C64.2, C65.2, C66.2
- net UUT_SCL: now reaches U37.6 (SCL2)
- net UUT_SDA: now reaches U37.7 (SDA2)
- net +5V: now reaches U37.8 (VDD2)
- net +5V: now also U35.8 (VDD2), U36.8 (VCC2), U38.20 (V_{DD2}), C63.1, C64.1, C65.1, C66.1
- net UUT_CIPO: now reaches U38.16 (SO)
- net UUT_COPI: now reaches U38.17 (SI)
- net UUT_SCK: now reaches U38.18 (SCLK)
- net SPI_SCK: now reaches U38.3 (MCLK)
- net SPI_COPI: now reaches U38.4 (MO)
- net SPI_CIPO: now reaches U38.5 (MI)
- net CAN_RX: now reaches U36.2 (RXD)
- net CAN_TX: now reaches U36.3 (TXD)
- net UUT_CAN_L: now reaches U36.6 (CANL)
- net UUT_CAN_H: now reaches U36.7 (CANH)
- net USART_MCU_RX: now reaches U35.2 (VOA)
- net USART_MCU_TX: now reaches U35.3 (VIB)
- net USART_UUT_RX: now reaches U35.6 (VOB)
- net USART_UUT_TX: now reaches U35.7 (VIA)
- no-connect marks 0 -> 8
Other:
- moved on the sheet: U35, U36, U37, U38
