File: io_expander_16.kicad_sch (KiCad schematic)
At the start: 2 parts, among them U30 PCA9555D

Commit message: first draft schematic?
Parts:
- C39: footprint (none) -> Capacitor_SMD:C_0603_1608Metric
Changed lines of the file:
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@@
       (effects (font (size 1.27 1.27)) (justify left))
     )
-    (property "Footprint" "" (id 2) (at 114.3 31.75 0)
+    (property "Footprint" "Capacitor_SMD:C_0603_1608Metric" (id 2) (at 114.3 31.75 0)
       (effects (font (size 1.27 1.27)) hide)
     )
