File: opto_isolation_8.kicad_sch (KiCad schematic)
At the start: 18 parts, among them U26 LTV-247, U27 LTV-247

Commit message: first draft schematic?
Parts:
- R10, R11, R12, R13, R14, R15, R16, R17, R18, R3, R4, R5, R6, R7, R8, R9: footprint (none) -> Resistor_SMD:R_0603_1608Metric
Changed lines of the file:
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@@
       (effects (font (size 1.27 1.27)) (justify left))
     )
-    (property "Footprint" "" (id 2) (at 81.28 92.71 0)
+    (property "Footprint" "Resistor_SMD:R_0603_1608Metric" (id 2) (at 81.28 92.71 0)
       (effects (font (size 1.27 1.27)) hide)
     )
@@
       (effects (font (size 1.27 1.27)) (justify left))
     )
-    (property "Footprint" "" (id 2) (at 81.28 54.61 0)
+    (property "Footprint" "Resistor_SMD:R_0603_1608Metric" (id 2) (at 81.28 54.61 0)
       (effects (font (size 1.27 1.27)) hide)
     )
@@
       (effects (font (size 1.27 1.27)) (justify left))
     )
-    (property "Footprint" "" (id 2) (at 81.28 143.51 0)
+    (property "Footprint" "Resistor_SMD:R_0603_1608Metric" (id 2) (at 81.28 143.51 0)
       (effects (font (size 1.27 1.27)) hide)
     )
@@
       (effects (font (size 1.27 1.27)) (justify left))
     )
-    (property "Footprint" "" (id 2) (at 170.18 154.94 0)
+    (property "Footprint" "Resistor_SMD:R_0603_1608Metric" (id 2) (at 170.18 154.94 0)
       (effects (font (size 1.27 1.27)) hide)
     )
@@
       (effects (font (size 1.27 1.27)) (justify left))
     )
-    (property "Footprint" "" (id 2) (at 160.02 154.94 0)
+    (property "Footprint" "Resistor_SMD:R_0603_1608Metric" (id 2) (at 160.02 154.94 0)
       (effects (font (size 1.27 1.27)) hide)
     )
@@
       (effects (font (size 1.27 1.27)) (justify left))
     )
-    (property "Footprint" "" (id 2) (at 129.54 154.94 0)
+    (property "Footprint" "Resistor_SMD:R_0603_1608Metric" (id 2) (at 129.54 154.94 0)
       (effects (font (size 1.27 1.27)) hide)
     )
@@
       (effects (font (size 1.27 1.27)) (justify left))
     )
-    (property "Footprint" "" (id 2) (at 139.7 154.94 0)
+    (property "Footprint" "Resistor_SMD:R_0603_1608Metric" (id 2) (at 139.7 154.94 0)
       (effects (font (size 1.27 1.27)) hide)
     )
@@
       (effects (font (size 1.27 1.27)) (justify left))
     )
-    (property "Footprint" "" (id 2) (at 180.34 154.94 0)
+    (property "Footprint" "Resistor_SMD:R_0603_1608Metric" (id 2) (at 180.34 154.94 0)
       (effects (font (size 1.27 1.27)) hide)
     )
@@
       (effects (font (size 1.27 1.27)) (justify left))
     )
-    (property "Footprint" "" (id 2) (at 81.28 105.41 0)
+    (property "Footprint" "Resistor_SMD:R_0603_1608Metric" (id 2) (at 81.28 105.41 0)
       (effects (font (size 1.27 1.27)) hide)
     )
@@
       (effects (font (size 1.27 1.27)) (justify left))
     )
-    (property "Footprint" "" (id 2) (at 119.38 154.94 0)
+    (property "Footprint" "Resistor_SMD:R_0603_1608Metric" (id 2) (at 119.38 154.94 0)
       (effects (font (size 1.27 1.27)) hide)
     )
@@
       (effects (font (size 1.27 1.27)) (justify left))
     )
-    (property "Footprint" "" (id 2) (at 81.28 80.01 0)
+    (property "Footprint" "Resistor_SMD:R_0603_1608Metric" (id 2) (at 81.28 80.01 0)
       (effects (font (size 1.27 1.27)) hide)
     )
@@
       (effects (font (size 1.27 1.27)) (justify left))
     )
-    (property "Footprint" "" (id 2) (at 81.28 67.31 0)
+    (property "Footprint" "Resistor_SMD:R_0603_1608Metric" (id 2) (at 81.28 67.31 0)
       (effects (font (size 1.27 1.27)) hide)
     )
@@
       (effects (font (size 1.27 1.27)) (justify left))
     )
-    (property "Footprint" "" (id 2) (at 81.28 130.81 0)
+    (property "Footprint" "Resistor_SMD:R_0603_1608Metric" (id 2) (at 81.28 130.81 0)
       (effects (font (size 1.27 1.27)) hide)
     )
@@
       (effects (font (size 1.27 1.27)) (justify left))
     )
-    (property "Footprint" "" (id 2) (at 81.28 118.11 0)
+    (property "Footprint" "Resistor_SMD:R_0603_1608Metric" (id 2) (at 81.28 118.11 0)
       (effects (font (size 1.27 1.27)) hide)
     )
@@
       (effects (font (size 1.27 1.27)) (justify left))
     )
-    (property "Footprint" "" (id 2) (at 149.86 154.94 0)
+    (property "Footprint" "Resistor_SMD:R_0603_1608Metric" (id 2) (at 149.86 154.94 0)
       (effects (font (size 1.27 1.27)) hide)
     )
@@
       (effects (font (size 1.27 1.27)) (justify left))
     )
-    (property "Footprint" "" (id 2) (at 109.22 154.94 0)
-      (effects (font (size 1.27 1.27)) hide)
-    )
+    (property "Footprint" "Resistor_SMD:R_0603_1608Metric" (id 2) (at 109.22 154.94 0)
+      (effects (font (size 1.27 1.27)) hide)
+    )
