File: test-kit-mcu.kicad_pcb (KiCad board)
At the start: 2 copper layers, 12 parts, among them J1 DIN41612_02x32_AB, J2 USB_B, U1 FT232RL, U2 ADuM121N, U3 STM32G473QET6, U4 MB85RS1MT, U5 ADR4525, U6 PGA113, U7 PGA113, U8 PGA113, U9 PGA113

Commit message: analog inputs, timer IO
Parts:
- added J3: Conn_02x32_Odd_Even, Connector_PinHeader_2.00mm:PinHeader_2x32_P2.00mm_Vertical, F.Cu at (97.0, 63.0)
- added PS1: MEE1S0503SC, Converter_DCDC:Converter_DCDC_Murata_MEE1SxxxxSC_THT, F.Cu at (469.7, 23.0)
- added U10: ADuM120N, Package_SO:SOIC-8_3.9x4.9mm_P1.27mm, F.Cu at (243.1, 110.2)
- added U11: ADuM120N, Package_SO:SOIC-8_3.9x4.9mm_P1.27mm, F.Cu at (234.6, 103.8)
- added U12: ADuM120N, Package_SO:SOIC-8_3.9x4.9mm_P1.27mm, F.Cu at (226.2, 103.8)
- added U13: ADuM120N, Package_SO:SOIC-8_3.9x4.9mm_P1.27mm, F.Cu at (234.6, 116.7)
- added U14: ADuM120N, Package_SO:SOIC-8_3.9x4.9mm_P1.27mm, F.Cu at (226.2, 116.7)
- added U15: ADuM120N, Package_SO:SOIC-8_3.9x4.9mm_P1.27mm, F.Cu at (234.6, 110.2)
- added U16: ADuM120N, Package_SO:SOIC-8_3.9x4.9mm_P1.27mm, F.Cu at (226.2, 110.2)
- added U17: ADuM120N, Package_SO:SOIC-8_3.9x4.9mm_P1.27mm, F.Cu at (243.1, 103.8)
- added U18: ADuM120N, Package_SO:SOIC-8_3.9x4.9mm_P1.27mm, F.Cu at (243.1, 135.8)
- added U19: ADuM120N, Package_SO:SOIC-8_3.9x4.9mm_P1.27mm, F.Cu at (234.6, 129.3)
- added U20: ADuM120N, Package_SO:SOIC-8_3.9x4.9mm_P1.27mm, F.Cu at (226.2, 129.3)
- added U21: ADuM120N, Package_SO:SOIC-8_3.9x4.9mm_P1.27mm, F.Cu at (234.6, 142.2)
- added U22: ADuM120N, Package_SO:SOIC-8_3.9x4.9mm_P1.27mm, F.Cu at (226.2, 142.2)
- added U23: ADuM120N, Package_SO:SOIC-8_3.9x4.9mm_P1.27mm, F.Cu at (234.6, 135.8)
- added U24: ADuM120N, Package_SO:SOIC-8_3.9x4.9mm_P1.27mm, F.Cu at (226.2, 135.8)
- added U25: ADuM120N, Package_SO:SOIC-8_3.9x4.9mm_P1.27mm, F.Cu at (243.1, 129.3)
- added U26: LTV-247, Package_SO:SOP-16_4.4x10.4mm_P1.27mm, F.Cu at (278.7, 128.7)
- added U27: LTV-247, Package_SO:SOP-16_4.4x10.4mm_P1.27mm, F.Cu at (269.6, 128.7)
- added U28: LTV-247, Package_SO:SOP-16_4.4x10.4mm_P1.27mm, F.Cu at (305.4, 106.5)
- added U29: LTV-247, Package_SO:SOP-16_4.4x10.4mm_P1.27mm, F.Cu at (296.2, 106.5)
- added U30: PCA9555D, Package_SO:SOIC-24W_7.5x15.4mm_P1.27mm, F.Cu at (271.5, 109.0)
- added U31: AMC1100DWV, Package_SO:SOIC-8_7.5x5.85mm_P1.27mm, F.Cu at (431.8, 23.7)
- added U32: AMC1100DWV, Package_SO:SOIC-8_7.5x5.85mm_P1.27mm, F.Cu at (431.8, 31.1)
- added U33: AMC1100DWV, Package_SO:SOIC-8_7.5x5.85mm_P1.27mm, F.Cu at (431.8, 38.5)
- added U34: AMC1100DWV, Package_SO:SOIC-8_7.5x5.85mm_P1.27mm, F.Cu at (445.8, 23.7)
- added U35: ADuM121N, Package_SO:SOIC-8_3.9x4.9mm_P1.27mm, F.Cu at (488.4, 42.6)
- added U36: ISO1050DUB, Package_SO:SOP-8_6.62x9.15mm_P2.54mm, F.Cu at (490.7, 25.3)
- added U37: ADuM1250, Package_SO:SOIC-8_3.9x4.9mm_P1.27mm, F.Cu at (501.4, 23.2)
- added U38: ADuM3153, Package_SO:SSOP-20_5.3x7.2mm_P0.65mm, F.Cu at (489.4, 35.0)
- J1: value DIN41612_02x32_AB -> Conn_02x32_Odd_Even; footprint Connector_DIN:DIN41612_B_2x32_Female_Vertical_THT -> Connector_PinHeader_2.00mm:PinHeader_2x32_P2.00mm_Vertical
- U6, U7: value PGA113 -> CD4051B; footprint Package_SO:TSSOP-10_3x3mm_P0.5mm -> Package_SO:SO-16_5.3x10.2mm_P1.27mm
- U8: value PGA113 -> CD4052B; footprint Package_SO:TSSOP-10_3x3mm_P0.5mm -> Package_SO:SO-16_5.3x10.2mm_P1.27mm
- U9: value PGA113 -> LTV-247; footprint Package_SO:TSSOP-10_3x3mm_P0.5mm -> Package_SO:SOP-16_4.4x10.4mm_P1.27mm
- moved J1 283.8 mm to (379.0, 22.0)
- moved U8 269.4 mm to (458.0, 25.9)
- moved U9 261.4 mm to (443.4, 33.4)
- moved U7 261.4 mm to (444.0, 45.2)
- moved U4 247.0 mm to (416.2, 23.2)
- moved U6 246.6 mm to (430.0, 48.1)
- moved U2 84.3 mm to (140.0, 70.0), turned to 90 degrees
- moved U1 68.9 mm to (140.0, 60.0), turned to 90 degrees
- moved J2 63.4 mm to (143.7, 51.1), turned to 180 degrees
- moved U5 37.5 mm to (147.0, 114.0), turned to 90 degrees
- moved U3 31.4 mm to (140.0, 90.0)
Connections:
- net /MCU/AI4_3 renamed /MCU/AI4_P
- net /MCU/AI4_4 renamed /MCU/AI4_N
- net /MCU/AI5_8 renamed /MCU/USB_RX
- net /MCU/SPI1_CIPO renamed Net-(U3-Pad85)
- net /MCU/SPI1_COPI renamed Net-(U3-Pad86)
- net /MCU/SPI1_SCK renamed Net-(U3-Pad84)
- U3 pad 1: unconnected-(U3-Pad1) -> /MCU/DO_2
- U3 pad 10: /MCU/DO_3 -> unconnected-(U3-Pad10)
- U3 pad 103: unconnected-(U3-Pad103) -> Net-(U3-Pad103)
- U3 pad 11: /MCU/DO_4 -> unconnected-(U3-Pad11)
- U3 pad 122: /MCU/I2C1_SDA -> unconnected-(U3-Pad122)
- U3 pad 123: /MCU/I2C1_SCL -> unconnected-(U3-Pad123)
- U3 pad 125: /MCU/USART1_TX -> /MCU/DO_0
- U3 pad 126: /MCU/USART1_RX -> /MCU/DO_1
- U3 pad 14: /MCU/DO_5 -> unconnected-(U3-Pad14)
- U3 pad 15: /MCU/DO_7 -> unconnected-(U3-Pad15)
- U3 pad 16: /MCU/DO_8 -> unconnected-(U3-Pad16)
- U3 pad 17: /MCU/DO_9 -> unconnected-(U3-Pad17)
- U3 pad 18: /MCU/DO_10 -> unconnected-(U3-Pad18)
- U3 pad 19: /MCU/DO_0 -> unconnected-(U3-Pad19)
- U3 pad 2: unconnected-(U3-Pad2) -> /MCU/DO_3
- U3 pad 20: /MCU/DO_1 -> unconnected-(U3-Pad20)
- U3 pad 26: /MCU/DO_2 -> unconnected-(U3-Pad26)
- U3 pad 3: unconnected-(U3-Pad3) -> /MCU/DO_4
- U3 pad 4: /MCU/SPI4_CIPO -> /MCU/DO_5
- U3 pad 48: /MCU/DO_11 -> unconnected-(U3-Pad48)
- U3 pad 49: /MCU/DO_12 -> unconnected-(U3-Pad49)
- U3 pad 5: /MCU/SPI4_COPI -> /MCU/DO_6
- U3 pad 50: /MCU/DO_13 -> unconnected-(U3-Pad50)
- U3 pad 51: /MCU/DO_14 -> INT_I2C_SDA
- U3 pad 52: /MCU/DO_15 -> INT_I2C_SCL
- U3 pad 53: unconnected-(U3-Pad53) -> /MCU/DO_7
- U3 pad 54: /MCU/AI5_3 -> /MCU/DO_8
- U3 pad 55: unconnected-(U3-Pad55) -> /MCU/DO_9
- U3 pad 56: /MCU/AI5_6 -> /MCU/DO_10
- U3 pad 57: /MCU/AI5_7 -> /MCU/DO_11
- U3 pad 58: /MCU/SPI4_SCK -> /MCU/DO_12
- U3 pad 59: unconnected-(U3-Pad59) -> /MCU/DO_13
- U3 pad 60: /MCU/AI4_1 -> /MCU/DO_14
- U3 pad 61: /MCU/AI4_2 -> /MCU/DO_15
- U3 pad 62: unconnected-(U3-Pad62) -> /MCU/USB_TX
- U3 pad 70: /MCU/AI4_5 -> unconnected-(U3-Pad70)
- U3 pad 71: /MCU/AI4_6 -> unconnected-(U3-Pad71)
- U3 pad 73: /MCU/AI5_5 -> unconnected-(U3-Pad73)
- U3 pad 74: /MCU/AI5_9 -> unconnected-(U3-Pad74)
- U3 pad 97: /MCU/DO_6 -> unconnected-(U3-Pad97)
- U4 pad 1: GND -> Net-(U3-Pad103)
- U6 pad 1: unconnected-(U6-Pad1) -> /Analogue Buffers/AI_S_4
- U6 pad 10: unconnected-(U6-Pad10) -> /Analogue Buffers/MUX_B
- U6 pad 2: unconnected-(U6-Pad2) -> /Analogue Buffers/AI_S_6
- U6 pad 3: unconnected-(U6-Pad3) -> Net-(R35-Pad1)
- U6 pad 4: unconnected-(U6-Pad4) -> /Analogue Buffers/AI_S_7
- U6 pad 5: unconnected-(U6-Pad5) -> /Analogue Buffers/AI_S_5
- U6 pad 7: unconnected-(U6-Pad7) -> GND1
- U6 pad 8: unconnected-(U6-Pad8) -> GND1
- U6 pad 9: unconnected-(U6-Pad9) -> /Analogue Buffers/MUX_C
- U7 pad 1: unconnected-(U7-Pad1) -> /Analogue Buffers/AI_S_12
- U7 pad 10: unconnected-(U7-Pad10) -> /Analogue Buffers/MUX_B
- U7 pad 2: unconnected-(U7-Pad2) -> /Analogue Buffers/AI_S_14
- U7 pad 3: unconnected-(U7-Pad3) -> Net-(R36-Pad1)
- U7 pad 4: unconnected-(U7-Pad4) -> /Analogue Buffers/AI_S_15
- U7 pad 5: unconnected-(U7-Pad5) -> /Analogue Buffers/AI_S_13
- U7 pad 7: unconnected-(U7-Pad7) -> GND1
- U7 pad 8: unconnected-(U7-Pad8) -> GND1
- U7 pad 9: unconnected-(U7-Pad9) -> /Analogue Buffers/MUX_C
- U8 pad 1: unconnected-(U8-Pad1) -> /Analogue Buffers/AI_F_4
- U8 pad 10: unconnected-(U8-Pad10) -> /Analogue Buffers/MUX_A
- U8 pad 2: unconnected-(U8-Pad2) -> /Analogue Buffers/AI_F_6
- U8 pad 3: unconnected-(U8-Pad3) -> Net-(R42-Pad1)
- U8 pad 4: unconnected-(U8-Pad4) -> /Analogue Buffers/AI_F_7
- U8 pad 5: unconnected-(U8-Pad5) -> /Analogue Buffers/AI_F_5
- U8 pad 7: unconnected-(U8-Pad7) -> GND1
- U8 pad 8: unconnected-(U8-Pad8) -> GND1
- U8 pad 9: unconnected-(U8-Pad9) -> /Analogue Buffers/MUX_B
- U9 pad 1: unconnected-(U9-Pad1) -> Net-(R46-Pad2)
- U9 pad 10: unconnected-(U9-Pad10) -> (no net)
- U9 pad 2: unconnected-(U9-Pad2) -> GND
- U9 pad 3: unconnected-(U9-Pad3) -> Net-(R47-Pad2)
- U9 pad 4: unconnected-(U9-Pad4) -> GND
- U9 pad 5: unconnected-(U9-Pad5) -> Net-(R48-Pad2)
- U9 pad 6: unconnected-(U9-Pad6) -> GND
- U9 pad 7: unconnected-(U9-Pad7) -> (no net)
- U9 pad 8: unconnected-(U9-Pad8) -> (no net)
- U9 pad 9: unconnected-(U9-Pad9) -> (no net)

Commit message: first draft schematic?
Parts:
- added C1: C_Small, Capacitor_SMD:C_0603_1608Metric, F.Cu at (411.2, 78.3)
- added C10: C_Small, Capacitor_SMD:C_0603_1608Metric, F.Cu at (486.7, 80.8)
- added C11: C_Small, Capacitor_SMD:C_0603_1608Metric, F.Cu at (482.7, 78.3)
- added C12: C_Small, Capacitor_SMD:C_0603_1608Metric, F.Cu at (482.7, 73.3)
- added C13: C_Small, Capacitor_SMD:C_0603_1608Metric, F.Cu at (494.7, 75.8)
- added C14: C_Small, Capacitor_SMD:C_0603_1608Metric, F.Cu at (494.7, 73.3)
- added C15: C_Small, Capacitor_SMD:C_0603_1608Metric, F.Cu at (490.7, 78.3)
- added C16: C_Small, Capacitor_SMD:C_0603_1608Metric, F.Cu at (486.7, 83.3)
- added C17: C_Small, Capacitor_SMD:C_0603_1608Metric, F.Cu at (486.7, 75.8)
- added C18: C_Small, Capacitor_SMD:C_0603_1608Metric, F.Cu at (482.7, 85.8)
- added C19: C_Small, Capacitor_SMD:C_0603_1608Metric, F.Cu at (482.7, 80.8)
- added C2: C_Small, Capacitor_SMD:C_0603_1608Metric, F.Cu at (403.2, 81.7)
- added C20: C_Small, Capacitor_SMD:C_0603_1608Metric, F.Cu at (486.7, 78.3)
- added C21: C_Small, Capacitor_SMD:C_0603_1608Metric, F.Cu at (482.7, 75.8)
- added C22: C_Small, Capacitor_SMD:C_0603_1608Metric, F.Cu at (490.7, 73.3)
- added C23: C_Small, Capacitor_SMD:C_0603_1608Metric, F.Cu at (436.7, 151.4)
- added C24: C_Small, Capacitor_SMD:C_0603_1608Metric, F.Cu at (444.8, 143.9)
- added C25: C_Small, Capacitor_SMD:C_0603_1608Metric, F.Cu at (440.7, 141.3)
- added C26: C_Small, Capacitor_SMD:C_0603_1608Metric, F.Cu at (440.7, 148.9)
- added C27: C_Small, Capacitor_SMD:C_0603_1608Metric, F.Cu at (436.7, 146.4)
- added C28: C_Small, Capacitor_SMD:C_0603_1608Metric, F.Cu at (436.7, 141.3)
- added C29: C_Small, Capacitor_SMD:C_0603_1608Metric, F.Cu at (448.8, 143.9)
- added C3: C_Small, Capacitor_SMD:C_0603_1608Metric, F.Cu at (410.9, 73.3)
- added C30: C_Small, Capacitor_SMD:C_0603_1608Metric, F.Cu at (448.8, 141.3)
- added C31: C_Small, Capacitor_SMD:C_0603_1608Metric, F.Cu at (444.8, 146.4)
- added C32: C_Small, Capacitor_SMD:C_0603_1608Metric, F.Cu at (440.7, 151.4)
- added C33: C_Small, Capacitor_SMD:C_0603_1608Metric, F.Cu at (440.7, 143.9)
- added C34: C_Small, Capacitor_SMD:C_0603_1608Metric, F.Cu at (436.7, 153.9)
- added C35: C_Small, Capacitor_SMD:C_0603_1608Metric, F.Cu at (436.7, 148.9)
- added C36: C_Small, Capacitor_SMD:C_0603_1608Metric, F.Cu at (440.7, 146.4)
- added C37: C_Small, Capacitor_SMD:C_0603_1608Metric, F.Cu at (436.7, 143.9)
- added C38: C_Small, Capacitor_SMD:C_0603_1608Metric, F.Cu at (444.8, 141.3)
- added C39: C_Small, Capacitor_SMD:C_0603_1608Metric, F.Cu at (502.6, 73.3)
- added C4: C_Small, Capacitor_SMD:C_0603_1608Metric, F.Cu at (403.2, 86.7)
- added C40: CE_10uF_16V, Capacitor_SMD:CP_Elec_4x5.3, F.Cu at (405.1, 75.0)
- added C41: C_Small, Capacitor_SMD:C_0603_1608Metric, F.Cu at (375.8, 143.9)
- added C42: C_Small, Capacitor_SMD:C_0603_1608Metric, F.Cu at (371.8, 141.3)
- added C43: C_Small, Capacitor_SMD:C_0603_1608Metric, F.Cu at (375.8, 141.3)
- added C44: C_Small, Capacitor_SMD:C_0603_1608Metric, F.Cu at (371.8, 151.4)
- added C45: C_0603_10%_10pF, Capacitor_SMD:C_0603_1608Metric, F.Cu at (371.8, 143.9)
- added C46: C_Small, Capacitor_SMD:C_0603_1608Metric, F.Cu at (367.8, 141.3)
- added C47: C_Small, Capacitor_SMD:C_0603_1608Metric, F.Cu at (367.8, 161.4)
- added C48: C_Small, Capacitor_SMD:C_0603_1608Metric, F.Cu at (375.8, 151.4)
- added C49: C_0603_10%_10pF, Capacitor_SMD:C_0603_1608Metric, F.Cu at (394.2, 73.3)
- added C5: C_Small, Capacitor_SMD:C_0603_1608Metric, F.Cu at (410.9, 75.8)
- added C50: C_0603_10%_10pF, Capacitor_SMD:C_0603_1608Metric, F.Cu at (376.5, 89.4)
- added C51: C_Small, Capacitor_SMD:C_0603_1608Metric, F.Cu at (371.8, 148.9)
- added C52: C_Small, Capacitor_SMD:C_0603_1608Metric, F.Cu at (375.8, 148.9)
- added C53: C_Small, Capacitor_SMD:C_0603_1608Metric, F.Cu at (367.8, 146.4)
- added C54: C_Small, Capacitor_SMD:C_0603_1608Metric, F.Cu at (367.8, 143.9)
- added C55: C_Small, Capacitor_SMD:C_0603_1608Metric, F.Cu at (383.9, 146.4)
- added C56: C_Small, Capacitor_SMD:C_0603_1608Metric, F.Cu at (387.9, 146.4)
- added C57: C_Small, Capacitor_SMD:C_0603_1608Metric, F.Cu at (371.8, 161.4)
- added C58: C_Small, Capacitor_SMD:C_0603_1608Metric, F.Cu at (367.8, 163.9)
- added C59: C_Small, Capacitor_SMD:C_0603_1608Metric, F.Cu at (453.5, 80.8)
- added C6: C_Small, Capacitor_SMD:C_0603_1608Metric, F.Cu at (407.2, 79.2)
- added C60: C_Small, Capacitor_SMD:C_0603_1608Metric, F.Cu at (453.5, 73.3)
- added C61: C_Small, Capacitor_SMD:C_0603_1608Metric, F.Cu at (453.5, 83.3)
- added C62: C_Small, Capacitor_SMD:C_0603_1608Metric, F.Cu at (457.5, 75.8)
- added C63: C_Small, Capacitor_SMD:C_0603_1608Metric, F.Cu at (457.5, 73.3)
- added C64: C_Small, Capacitor_SMD:C_0603_1608Metric, F.Cu at (453.5, 75.8)
- added C65: C_Small, Capacitor_SMD:C_0603_1608Metric, F.Cu at (453.5, 78.3)
- added C66: C_Small, Capacitor_SMD:C_0603_1608Metric, F.Cu at (457.5, 78.3)
- added C67: C_Small, Capacitor_SMD:C_0603_1608Metric, F.Cu at (439.2, 82.3)
- added C68: C_Small, Capacitor_SMD:C_0603_1608Metric, F.Cu at (426.3, 95.2)
- added C69: C_Small, Capacitor_SMD:C_0603_1608Metric, F.Cu at (430.7, 86.2)
- added C7: C_Small, Capacitor_SMD:C_0603_1608Metric, F.Cu at (482.7, 83.3)
- added C70: C_Small, Capacitor_SMD:C_0603_1608Metric, F.Cu at (426.3, 92.7)
- added C71: C_Small, Capacitor_SMD:C_0603_1608Metric, F.Cu at (434.8, 86.2)
- added C72: C_Small, Capacitor_SMD:C_0603_1608Metric, F.Cu at (430.7, 88.7)
- added C73: C_Small, Capacitor_SMD:C_0603_1608Metric, F.Cu at (422.3, 95.2)
- added C74: C_Small, Capacitor_SMD:C_0603_1608Metric, F.Cu at (422.3, 97.7)
- added C75: C_Small, Capacitor_SMD:C_0603_1608Metric, F.Cu at (422.3, 92.7)
- added C76: C_Small, Capacitor_SMD:C_0603_1608Metric, F.Cu at (443.2, 79.8)
- added C77: C_Small, Capacitor_SMD:C_0603_1608Metric, F.Cu at (439.2, 79.8)
- added C78: C_Small, Capacitor_SMD:C_0603_1608Metric, F.Cu at (430.7, 91.2)
- added C8: C_Small, Capacitor_SMD:C_0603_1608Metric, F.Cu at (490.7, 75.8)
- added C9: C_Small, Capacitor_SMD:C_0603_1608Metric, F.Cu at (486.7, 73.3)
- added D2: LED_Small, LED_SMD:LED_0603_1608Metric, F.Cu at (376.6, 81.8)
- added D3: LED_Small, LED_SMD:LED_0603_1608Metric, F.Cu at (382.2, 75.9)
- added D4: LED_Small, LED_SMD:LED_0603_1608Metric, F.Cu at (372.5, 81.8)
- added D5: LED_Small, LED_SMD:LED_0603_1608Metric, F.Cu at (372.5, 87.0)
- added D6: LED_Small, LED_SMD:LED_0603_1608Metric, F.Cu at (367.9, 133.2)
- added D7: LED_Small, LED_SMD:LED_0603_1608Metric, F.Cu at (386.2, 73.3)
- added D8: LED_Small, LED_SMD:LED_0603_1608Metric, F.Cu at (382.2, 73.3)
- added D9: LED_Small, LED_SMD:LED_0603_1608Metric, F.Cu at (372.5, 84.4)
- added FB1: FerriteBead_Small, Inductor_SMD:L_0603_1608Metric, F.Cu at (403.2, 84.2)
- added J4: Conn_02x16_Odd_Even, Connector_PinHeader_2.00mm:PinHeader_2x32_P2.00mm_Horizontal, F.Cu at (110.0, 34.1)
- added J5: Conn_02x16_Odd_Even, Connector_PinHeader_2.00mm:PinHeader_2x32_P2.00mm_Horizontal, F.Cu at (168.0, 114.9)
- added J6: Conn_ARM_JTAG_SWD_10, Connector_PinHeader_1.27mm:PinHeader_2x05_P1.27mm_Vertical_SMD, F.Cu at (375.3, 76.3)
- added J7: Conn_01x10, Connector_PinHeader_2.54mm:PinHeader_1x10_P2.54mm_Vertical, F.Cu at (368.1, 74.4)
- added J8: Conn_01x10, Connector_PinHeader_2.54mm:PinHeader_1x10_P2.54mm_Vertical, F.Cu at (368.1, 101.9)
- added L1: L_4.7uH_800mA_82472C, Inductor_SMD:L_0603_1608Metric, F.Cu at (407.2, 81.7)
- added R1: R, Resistor_SMD:R_0603_1608Metric, F.Cu at (403.2, 79.2)
- added R10: R_Small, Resistor_SMD:R_0603_1608Metric, F.Cu at (400.9, 141.3)
- added R11: R_Small, Resistor_SMD:R_0603_1608Metric, F.Cu at (400.9, 151.4)
- added R12: R_Small, Resistor_SMD:R_0603_1608Metric, F.Cu at (396.9, 151.4)
- added R13: R_Small, Resistor_SMD:R_0603_1608Metric, F.Cu at (404.9, 141.3)
- added R14: R_Small, Resistor_SMD:R_0603_1608Metric, F.Cu at (396.9, 148.9)
- added R15: R_Small, Resistor_SMD:R_0603_1608Metric, F.Cu at (408.9, 143.9)
- added R16: R_Small, Resistor_SMD:R_0603_1608Metric, F.Cu at (400.9, 143.9)
- added R17: R_Small, Resistor_SMD:R_0603_1608Metric, F.Cu at (396.9, 146.4)
- added R18: R_Small, Resistor_SMD:R_0603_1608Metric, F.Cu at (400.9, 146.4)
- added R19: R_Small, Resistor_SMD:R_0603_1608Metric, F.Cu at (416.8, 143.9)
- added R2: R, Resistor_SMD:R_0603_1608Metric, F.Cu at (414.9, 73.3)
- added R20: R_Small, Resistor_SMD:R_0603_1608Metric, F.Cu at (420.8, 148.9)
- added R21: R_Small, Resistor_SMD:R_0603_1608Metric, F.Cu at (428.8, 141.3)
- added R22: R_Small, Resistor_SMD:R_0603_1608Metric, F.Cu at (416.8, 141.3)
- added R23: R_Small, Resistor_SMD:R_0603_1608Metric, F.Cu at (424.8, 143.9)
- added R24: R_Small, Resistor_SMD:R_0603_1608Metric, F.Cu at (416.8, 153.9)
- added R25: R_Small, Resistor_SMD:R_0603_1608Metric, F.Cu at (424.8, 146.4)
- added R26: R_Small, Resistor_SMD:R_0603_1608Metric, F.Cu at (420.8, 141.3)
- added R27: R_Small, Resistor_SMD:R_0603_1608Metric, F.Cu at (420.8, 151.4)
- added R28: R_Small, Resistor_SMD:R_0603_1608Metric, F.Cu at (416.8, 151.4)
- added R29: R_Small, Resistor_SMD:R_0603_1608Metric, F.Cu at (424.8, 141.3)
- added R3: R_Small, Resistor_SMD:R_0603_1608Metric, F.Cu at (396.9, 143.9)
- added R30: R_Small, Resistor_SMD:R_0603_1608Metric, F.Cu at (416.8, 148.9)
- added R31: R_Small, Resistor_SMD:R_0603_1608Metric, F.Cu at (428.8, 143.9)
- added R32: R_Small, Resistor_SMD:R_0603_1608Metric, F.Cu at (420.8, 143.9)
- added R33: R_Small, Resistor_SMD:R_0603_1608Metric, F.Cu at (416.8, 146.4)
- added R34: R_Small, Resistor_SMD:R_0603_1608Metric, F.Cu at (420.8, 146.4)
- added R35: R_0603_1%_820k, Resistor_SMD:R_0603_1608Metric, F.Cu at (383.9, 148.9)
- added R36: R_Small, Resistor_SMD:R_0603_1608Metric, F.Cu at (375.8, 156.4)
- added R37: R_Small, Resistor_SMD:R_0603_1608Metric, F.Cu at (371.8, 158.9)
- added R38: R_0603_1%_200k, Resistor_SMD:R_0603_1608Metric, F.Cu at (367.8, 153.9)
- added R39: R_Small, Resistor_SMD:R_0603_1608Metric, F.Cu at (367.8, 158.9)
- added R4: R_Small, Resistor_SMD:R_0603_1608Metric, F.Cu at (400.9, 148.9)
- added R40: R_Small, Resistor_SMD:R_0603_1608Metric, F.Cu at (387.9, 143.9)
- added R41: R_Small, Resistor_SMD:R_0603_1608Metric, F.Cu at (367.8, 151.4)
- added R42: R_Small, Resistor_SMD:R_0603_1608Metric, F.Cu at (379.9, 146.4)
- added R43: R_Small, Resistor_SMD:R_0603_1608Metric, F.Cu at (387.9, 141.3)
- added R44: R_Small, Resistor_SMD:R_0603_1608Metric, F.Cu at (367.8, 156.4)
- added R45: R_Small, Resistor_SMD:R_0603_1608Metric, F.Cu at (379.9, 151.4)
- added R46: R_Small, Resistor_SMD:R_0603_1608Metric, F.Cu at (371.8, 146.4)
- added R47: R_Small, Resistor_SMD:R_0603_1608Metric, F.Cu at (367.8, 148.9)
- added R48: R_Small, Resistor_SMD:R_0603_1608Metric, F.Cu at (383.9, 143.9)
- added R49: R_0603_1%_100R, Resistor_SMD:R_0603_1608Metric, F.Cu at (379.9, 148.9)
- added R5: R_Small, Resistor_SMD:R_0603_1608Metric, F.Cu at (408.9, 141.3)
- added R50: R_0R_NNF, Resistor_SMD:R_0603_1608Metric, F.Cu at (382.1, 78.5)
- added R51: R_Small, Resistor_SMD:R_0603_1608Metric, F.Cu at (371.8, 153.9)
- added R52: R_Small, Resistor_SMD:R_0603_1608Metric, F.Cu at (375.8, 146.4)
- added R53: R_Small, Resistor_SMD:R_0603_1608Metric, F.Cu at (383.9, 141.3)
- added R54: R_Small, Resistor_SMD:R_0603_1608Metric, F.Cu at (379.9, 143.9)
- added R55: R_Small, Resistor_SMD:R_0603_1608Metric, F.Cu at (379.9, 141.3)
- added R56: R_Small, Resistor_SMD:R_0603_1608Metric, F.Cu at (375.8, 153.9)
- added R57: R_0R_NNF, Resistor_SMD:R_0603_1608Metric, F.Cu at (390.2, 75.8)
- added R58: R_0R_NNF, Resistor_SMD:R_0603_1608Metric, F.Cu at (372.5, 89.5)
- added R59: R_Small, Resistor_SMD:R_0603_1608Metric, F.Cu at (376.5, 84.3)
- added R6: R_Small, Resistor_SMD:R_0603_1608Metric, F.Cu at (396.9, 141.3)
- added R60: R_Small, Resistor_SMD:R_0603_1608Metric, F.Cu at (382.1, 81.0)
- added R61: R_Small, Resistor_SMD:R_0603_1608Metric, F.Cu at (375.5, 92.0)
- added R62: R_Small, Resistor_SMD:R_0603_1608Metric, F.Cu at (376.5, 86.8)
- added R63: R_Small, Resistor_SMD:R_0603_1608Metric, F.Cu at (380.5, 84.3)
- added R64: R_Small, Resistor_SMD:R_0603_1608Metric, F.Cu at (386.2, 75.9)
- added R65: R_Small, Resistor_SMD:R_0603_1608Metric, F.Cu at (380.5, 86.8)
- added R66: R_Small, Resistor_SMD:R_0603_1608Metric, F.Cu at (390.2, 73.3)
- added R67: R_0603_1%_100R, Resistor_SMD:R_0603_1608Metric, F.Cu at (371.8, 156.4)
- added R7: R_Small, Resistor_SMD:R_0603_1608Metric, F.Cu at (404.9, 143.9)
- added R8: R_Small, Resistor_SMD:R_0603_1608Metric, F.Cu at (396.9, 153.9)
- added R9: R_Small, Resistor_SMD:R_0603_1608Metric, F.Cu at (404.9, 146.4)
- added U39: ADuM120N, Package_SO:SOIC-8_3.9x4.9mm_P1.27mm, F.Cu at (433.0, 81.7)
- added U40: ADuM120N, Package_SO:SOIC-8_3.9x4.9mm_P1.27mm, F.Cu at (441.4, 75.3)
- added U41: ADuM120N, Package_SO:SOIC-8_3.9x4.9mm_P1.27mm, F.Cu at (424.5, 88.2)
- added U42: ADuM120N, Package_SO:SOIC-8_3.9x4.9mm_P1.27mm, F.Cu at (424.5, 81.7)
- added U43: ADuM120N, Package_SO:SOIC-8_3.9x4.9mm_P1.27mm, F.Cu at (433.0, 75.3)
- added U44: ADR4530, Package_SO:SOIC-8_3.9x4.9mm_P1.27mm, F.Cu at (470.7, 75.3)
- added Y1: CRYSTAL_8MHZ_ABM3-8.000MHZ-D2Y-T, Crystal:Crystal_SMD_Abracon_ABM3-2Pin_5.0x3.2mm, F.Cu at (369.6, 129.5)
- J1, J3: value Conn_02x32_Odd_Even -> Conn_02x16_Odd_Even; footprint Connector_PinHeader_2.00mm:PinHeader_2x32_P2.00mm_Vertical -> Connector_PinHeader_2.00mm:PinHeader_2x32_P2.00mm_Horizontal
- U5: value ADR4525 -> ADuM120N
- moved J1 293.1 mm to (101.0, 114.9), turned to -90 degrees
- moved U5 280.2 mm to (424.5, 75.3), turned to 0 degrees
- moved J2 115.3 mm to (29.4, 65.5), turned to -90 degrees
- moved PS1 109.3 mm to (360.9, 12.3)
- moved U31 109.3 mm to (323.0, 13.0)
- moved U32 109.3 mm to (323.0, 20.4)
- moved U33 109.3 mm to (323.0, 27.8)
- moved U34 109.3 mm to (337.0, 13.0)
- moved U35 109.3 mm to (379.6, 32.0)
- moved U36 109.3 mm to (381.9, 14.6)
- moved U37 109.3 mm to (392.6, 12.5)
- moved U38 109.3 mm to (380.6, 24.4)
- moved U4 109.3 mm to (307.4, 12.5)
- moved U8 109.3 mm to (349.2, 15.2)
- moved U9 109.3 mm to (334.6, 22.7)
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Connections:
- net /Analogue Buffers/MUX_A renamed /Analogue Inputs/MUX_A
- net /Analogue Buffers/MUX_B renamed /Analogue Inputs/MUX_B
- net /Analogue Buffers/MUX_C renamed /Analogue Inputs/MUX_C
- J1 pad 10: unconnected-(J1-Pad10) -> /AI_S_10
- J1 pad 11: unconnected-(J1-Pad11) -> /AI_S_3
- J1 pad 12: unconnected-(J1-Pad12) -> /AI_S_11
- J1 pad 13: unconnected-(J1-Pad13) -> /AI_S_4
- J1 pad 14: unconnected-(J1-Pad14) -> /AI_S_12
- J1 pad 15: unconnected-(J1-Pad15) -> /AI_S_5
- J1 pad 16: Net-(J1-Pad16) -> GND1
- J1 pad 17: unconnected-(J1-Pad17) -> /AI_S_6
- J1 pad 18: unconnected-(J1-Pad18) -> /AI_S_13
- J1 pad 19: unconnected-(J1-Pad19) -> /AI_S_7
- J1 pad 20: unconnected-(J1-Pad20) -> /AI_S_14
- J1 pad 21: Net-(J1-Pad21) -> GND1
- J1 pad 22: unconnected-(J1-Pad22) -> /AI_S_15
- J1 pad 23: unconnected-(J1-Pad23) -> /AI_F_0
- J1 pad 24: unconnected-(J1-Pad24) -> /AI_F_4
- J1 pad 25: unconnected-(J1-Pad25) -> /AI_F_1
- J1 pad 26: unconnected-(J1-Pad26) -> /AI_F_5
- J1 pad 27: unconnected-(J1-Pad27) -> /AI_F_2
- J1 pad 28: Net-(J1-Pad16) -> GND1
- J1 pad 29: unconnected-(J1-Pad29) -> /AI_F_3
- J1 pad 3: unconnected-(J1-Pad3) -> /AI_S_0
- J1 pad 30: unconnected-(J1-Pad30) -> /AI_F_6
- J1 pad 31: unconnected-(J1-Pad31) -> GND1
- J1 pad 32: unconnected-(J1-Pad32) -> /AI_F_7
- J1 pad 33: Net-(J1-Pad21) -> (no net)
- J1 pad 34: unconnected-(J1-Pad34) -> (no net)
- J1 pad 35: unconnected-(J1-Pad35) -> (no net)
- J1 pad 36: unconnected-(J1-Pad36) -> (no net)
- J1 pad 37: unconnected-(J1-Pad37) -> (no net)
- J1 pad 38: unconnected-(J1-Pad38) -> (no net)
- J1 pad 39: unconnected-(J1-Pad39) -> (no net)
- J1 pad 4: Net-(J1-Pad16) -> GND1
- J1 pad 40: Net-(J1-Pad16) -> (no net)
- J1 pad 41: unconnected-(J1-Pad41) -> (no net)
- J1 pad 42: unconnected-(J1-Pad42) -> (no net)
- J1 pad 43: unconnected-(J1-Pad43) -> (no net)
- J1 pad 44: unconnected-(J1-Pad44) -> (no net)
- J1 pad 45: Net-(J1-Pad21) -> (no net)
- J1 pad 46: unconnected-(J1-Pad46) -> (no net)
- J1 pad 47: unconnected-(J1-Pad47) -> (no net)
- J1 pad 48: unconnected-(J1-Pad48) -> (no net)
- J1 pad 49: unconnected-(J1-Pad49) -> (no net)
- J1 pad 5: unconnected-(J1-Pad5) -> /AI_S_1
- J1 pad 50: unconnected-(J1-Pad50) -> (no net)
- J1 pad 51: unconnected-(J1-Pad51) -> (no net)
- J1 pad 52: Net-(J1-Pad16) -> (no net)
- J1 pad 53: unconnected-(J1-Pad53) -> (no net)
- J1 pad 54: unconnected-(J1-Pad54) -> (no net)
- J1 pad 55: unconnected-(J1-Pad55) -> (no net)
- J1 pad 56: unconnected-(J1-Pad56) -> (no net)
- J1 pad 57: Net-(J1-Pad21) -> (no net)
- J1 pad 58: unconnected-(J1-Pad58) -> (no net)
- J1 pad 59: unconnected-(J1-Pad59) -> (no net)
- J1 pad 6: unconnected-(J1-Pad6) -> /AI_S_8
- J1 pad 60: unconnected-(J1-Pad60) -> (no net)
- J1 pad 61: unconnected-(J1-Pad61) -> (no net)
- J1 pad 62: unconnected-(J1-Pad62) -> (no net)
- J1 pad 63: unconnected-(J1-Pad63) -> (no net)
- J1 pad 64: Net-(J1-Pad16) -> (no net)
- J1 pad 7: unconnected-(J1-Pad7) -> /AI_S_2
- J1 pad 8: unconnected-(J1-Pad8) -> /AI_S_9
- J1 pad 9: Net-(J1-Pad21) -> GND1
- J3 pad 10: /Digital IO/DI_F_2 -> /IC_3
- J3 pad 11: /Digital IO/DO_F_3 -> /PWM_4
- J3 pad 12: /Digital IO/DI_F_3 -> /IC_4
- J3 pad 13: /Digital IO/DO_F_4 -> /PWM_5
- J3 pad 14: /Digital IO/DI_F_4 -> unconnected-(J3-Pad14)
- J3 pad 15: /Digital IO/DO_F_5 -> /PWM_6
- J3 pad 17: /Digital IO/DO_F_6 -> /PWM_7
- J3 pad 18: /Digital IO/DI_F_5 -> unconnected-(J3-Pad18)
- J3 pad 19: /Digital IO/DO_F_7 -> unconnected-(J3-Pad19)
- J3 pad 20: /Digital IO/DI_F_6 -> unconnected-(J3-Pad20)
- J3 pad 22: /Digital IO/DI_F_7 -> /UUT_USART_RX
- J3 pad 23: /Digital IO/DO_F_8 -> /UUT_USART_TX
- J3 pad 24: /Digital IO/DI_F_8 -> /UUT_CAN_H
- J3 pad 25: /Digital IO/DO_F_9 -> /UUT_I2C_SCL
- J3 pad 26: /Digital IO/DI_F_9 -> /UUT_CAN_L
- J3 pad 27: /Digital IO/DO_F_10 -> /UUT_I2C_SDA
- J3 pad 29: /Digital IO/DO_F_11 -> /UUT_SPI_SCK
- J3 pad 3: /Digital IO/DO_F_0 -> /PWM_1
- J3 pad 30: /Digital IO/DI_F_10 -> /UUT_SPI_COPI
- J3 pad 31: /Digital IO/DO_F_12 -> GND1
- J3 pad 32: /Digital IO/DI_F_11 -> /UUT_SPI_CIPO
- J3 pad 33: GND1 -> (no net)
- J3 pad 34: /Digital IO/DI_F_12 -> (no net)
- J3 pad 35: /Digital IO/DO_F_13 -> (no net)
- J3 pad 36: /Digital IO/DI_F_13 -> (no net)
- J3 pad 37: /Digital IO/DO_F_14 -> (no net)
- J3 pad 38: /Digital IO/DI_F_14 -> (no net)
- J3 pad 39: /Digital IO/DO_F_15 -> (no net)
- J3 pad 40: GND1 -> (no net)
- J3 pad 41: /Digital IO/DO_S_0 -> (no net)
- J3 pad 42: /Digital IO/DI_F_15 -> (no net)
- J3 pad 43: /Digital IO/DO_S_1 -> (no net)
- J3 pad 44: /Digital IO/DI_S_0 -> (no net)
- J3 pad 45: GND1 -> (no net)
- J3 pad 46: /Digital IO/DI_S_1 -> (no net)
- J3 pad 47: /Digital IO/DO_S_2 -> (no net)
- J3 pad 48: /Digital IO/DI_S_2 -> (no net)
- J3 pad 49: /Digital IO/DO_S_3 -> (no net)
- J3 pad 5: /Digital IO/DO_F_1 -> /PWM_2
- J3 pad 50: /Digital IO/DI_S_3 -> (no net)
- J3 pad 51: /Digital IO/DO_S_4 -> (no net)
- J3 pad 52: GND1 -> (no net)
- J3 pad 53: /Digital IO/DO_S_5 -> (no net)
- J3 pad 54: /Digital IO/DI_S_4 -> (no net)
- J3 pad 55: /Digital IO/DO_S_6 -> (no net)
- J3 pad 56: /Digital IO/DI_S_5 -> (no net)
- J3 pad 57: GND1 -> (no net)
- J3 pad 58: /Digital IO/DI_S_6 -> (no net)
- J3 pad 59: /Digital IO/DO_S_7 -> (no net)
- J3 pad 6: /Digital IO/DI_F_0 -> /IC_1
- J3 pad 60: /Digital IO/DI_S_7 -> (no net)
- J3 pad 61: unconnected-(J3-Pad61) -> (no net)
- J3 pad 62: unconnected-(J3-Pad62) -> (no net)
- J3 pad 63: unconnected-(J3-Pad63) -> (no net)
- J3 pad 64: GND1 -> (no net)
- J3 pad 7: /Digital IO/DO_F_2 -> /PWM_3
- J3 pad 8: /Digital IO/DI_F_1 -> /IC_2
- U10 pad 6: /Digital IO/DO_F_1 -> /DO_F_1
- U10 pad 7: /Digital IO/DO_F_0 -> /DO_F_0
- U11 pad 6: /Digital IO/DO_F_3 -> /DO_F_3
- U11 pad 7: /Digital IO/DO_F_2 -> /DO_F_2
- U12 pad 6: /Digital IO/DO_F_5 -> /DO_F_5
- U12 pad 7: /Digital IO/DO_F_4 -> /DO_F_4
- U13 pad 6: /Digital IO/DO_F_7 -> /DO_F_7
- U13 pad 7: /Digital IO/DO_F_6 -> /DO_F_6
- U14 pad 6: /Digital IO/DO_F_9 -> /DO_F_9
- U14 pad 7: /Digital IO/DO_F_8 -> /DO_F_8
- U15 pad 6: /Digital IO/DO_F_11 -> /DO_F_11
- U15 pad 7: /Digital IO/DO_F_10 -> /DO_F_10
- U16 pad 6: /Digital IO/DO_F_13 -> /DO_F_13
- U16 pad 7: /Digital IO/DO_F_12 -> /DO_F_12
- U17 pad 6: /Digital IO/DO_F_15 -> /DO_F_15
- U17 pad 7: /Digital IO/DO_F_14 -> /DO_F_14
- U18 pad 2: /Digital IO/DI_F_0 -> /DI_F_0
- U18 pad 3: /Digital IO/DI_F_1 -> /DI_F_1
- U19 pad 2: /Digital IO/DI_F_2 -> /DI_F_2
- U19 pad 3: /Digital IO/DI_F_3 -> /DI_F_3
- U2 pad 2: /USB/USB_TX -> /MCU/USB_RX
- U2 pad 3: /USB/USB_RX -> /MCU/USB_TX
- U20 pad 2: /Digital IO/DI_F_4 -> /DI_F_4
- U20 pad 3: /Digital IO/DI_F_5 -> /DI_F_5
- U21 pad 2: /Digital IO/DI_F_6 -> /DI_F_6
- U21 pad 3: /Digital IO/DI_F_7 -> /DI_F_7
- U22 pad 2: /Digital IO/DI_F_8 -> /DI_F_8
- U22 pad 3: /Digital IO/DI_F_9 -> /DI_F_9
- U23 pad 2: /Digital IO/DI_F_10 -> /DI_F_10
- U23 pad 3: /Digital IO/DI_F_11 -> /DI_F_11
- U24 pad 2: /Digital IO/DI_F_12 -> /DI_F_12
- U24 pad 3: /Digital IO/DI_F_13 -> /DI_F_13
- U25 pad 2: /Digital IO/DI_F_14 -> /DI_F_14
- U25 pad 3: /Digital IO/DI_F_15 -> /DI_F_15
- U26 pad 10: /Digital IO/Digital In Slow/VCC_OUT -> +12V
- U26 pad 11: /Digital IO/DO_S_2 -> /DO_S_2
- U26 pad 12: /Digital IO/Digital In Slow/VCC_OUT -> +12V
- U26 pad 13: /Digital IO/DO_S_1 -> /DO_S_1
- U26 pad 14: /Digital IO/Digital In Slow/VCC_OUT -> +12V
- U26 pad 15: /Digital IO/DO_S_0 -> /DO_S_0
- U26 pad 16: /Digital IO/Digital In Slow/VCC_OUT -> +12V
- U26 pad 9: /Digital IO/DO_S_3 -> /DO_S_3
- U27 pad 10: /Digital IO/Digital In Slow/VCC_OUT -> +12V
- U27 pad 11: /Digital IO/DO_S_6 -> /DO_S_6
- U27 pad 12: /Digital IO/Digital In Slow/VCC_OUT -> +12V
- U27 pad 13: /Digital IO/DO_S_5 -> /DO_S_5
- U27 pad 14: /Digital IO/Digital In Slow/VCC_OUT -> +12V
- U27 pad 15: /Digital IO/DO_S_4 -> /DO_S_4
- U27 pad 16: /Digital IO/Digital In Slow/VCC_OUT -> +12V
- U27 pad 9: /Digital IO/DO_S_7 -> /DO_S_7
- U3 pad 10: unconnected-(U3-Pad10) -> /MCU/SP_1
- U3 pad 104: unconnected-(U3-Pad104) -> /MCU/HW_2
- U3 pad 105: /MCU/I2C3_SCL -> /Comms/I2C_SCL
- U3 pad 106: /MCU/I2C3_SDA -> /Comms/I2C_SDA
- U3 pad 107: unconnected-(U3-Pad107) -> /MCU/HW_1
- U3 pad 108: /MCU/CAN1_RX -> /Comms/CAN_RX
- U3 pad 109: /MCU/CAN1_TX -> /Comms/CAN_TX
- U3 pad 11: unconnected-(U3-Pad11) -> /MCU/SP_2
- U3 pad 112: unconnected-(U3-Pad112) -> /MCU/LED_0
- U3 pad 113: /MCU/TIM2_1 -> /MCU/PWM_1
- U3 pad 114: /MCU/TIM2_2 -> /MCU/PWM_2
- U3 pad 115: unconnected-(U3-Pad115) -> /MCU/LED_1
- U3 pad 116: /MCU/TIM2_4 -> /MCU/PWM_4
- U3 pad 117: /MCU/TIM2_3 -> /MCU/PWM_3
- U3 pad 120: unconnected-(U3-Pad120) -> /MCU/SP_10
- U3 pad 121: unconnected-(U3-Pad121) -> /MCU/IC_1
- U3 pad 122: unconnected-(U3-Pad122) -> /MCU/IC_2
- U3 pad 123: unconnected-(U3-Pad123) -> /MCU/IC_3
- U3 pad 124: unconnected-(U3-Pad124) -> /MCU/IC_4
- U3 pad 14: unconnected-(U3-Pad14) -> /MCU/SP_3
- U3 pad 15: unconnected-(U3-Pad15) -> /MCU/SP_5
- U3 pad 16: unconnected-(U3-Pad16) -> /MCU/SP_6
- U3 pad 17: unconnected-(U3-Pad17) -> /MCU/SP_7
- U3 pad 18: unconnected-(U3-Pad18) -> /MCU/SP_8
- U3 pad 19: unconnected-(U3-Pad19) -> Net-(U3-Pad19)
- U3 pad 20: unconnected-(U3-Pad20) -> Net-(U3-Pad20)
- U3 pad 21: unconnected-(U3-Pad21) -> /MCU/HW_0
- U3 pad 26: unconnected-(U3-Pad26) -> /MCU/SP_0
- U3 pad 27: /MCU/AI1_1 -> /Analogue Inputs/ADC1_P
- U3 pad 28: /MCU/AI2_4 -> /Analogue Inputs/ADC1_N
- U3 pad 29: /MCU/USART2_TX -> /Comms/USART_MCU_TX
- U3 pad 32: /MCU/USART2_RX -> /Comms/USART_MCU_RX
- U3 pad 36: /MCU/AI2_3 -> /MCU/LED_6
- U3 pad 39: /MCU/AI1_4 -> /MCU/PWM_7
- U3 pad 40: /MCU/AI1_3 -> /MCU/PWM_8
- U3 pad 41: /MCU/AI2_1 -> /MCU/SP_9
- U3 pad 48: unconnected-(U3-Pad48) -> /Analogue Inputs/ADC_MUX_A
- U3 pad 49: unconnected-(U3-Pad49) -> /Analogue Inputs/ADC_MUX_B
- U3 pad 50: unconnected-(U3-Pad50) -> /Analogue Inputs/ADC_MUX_C
- U3 pad 66: /MCU/AI1_2 -> /MCU/SP_11
- U3 pad 67: /MCU/SPI2_SCK -> /Comms/SPI_SCK
- U3 pad 68: unconnected-(U3-Pad68) -> /MCU/PWM_5
- U3 pad 69: /MCU/AI2_2 -> /MCU/PWM_6
- U3 pad 70: unconnected-(U3-Pad70) -> /MCU/LED_2
- U3 pad 71: unconnected-(U3-Pad71) -> /MCU/LED_3
- U3 pad 72: /MCU/AI5_4 -> /MCU/LED_4
- U3 pad 73: unconnected-(U3-Pad73) -> /Analogue Inputs/ADC2_P
- U3 pad 74: unconnected-(U3-Pad74) -> /Analogue Inputs/ADC2_N
- U3 pad 75: /MCU/AI4_P -> /Analogue Inputs/ADC3_P
- U3 pad 76: /MCU/AI4_N -> /Analogue Inputs/ADC3_N
- U3 pad 77: unconnected-(U3-Pad77) -> /MCU/LED_5
- U3 pad 82: unconnected-(U3-Pad82) -> /MCU/SP_12
- U3 pad 83: unconnected-(U3-Pad83) -> /MCU/SP_13
- U3 pad 89: /MCU/AI5_1 -> /Analogue Inputs/ADC4_P
- U3 pad 90: /MCU/AI5_2 -> /Analogue Inputs/ADC4_N
- U3 pad 91: /MCU/SPI2_CIPO -> /Comms/SPI_CIPO
- U3 pad 92: /MCU/SPI2_COPI -> /Comms/SPI_COPI
- U3 pad 93: unconnected-(U3-Pad93) -> /MCU/LED_7
- U3 pad 97: unconnected-(U3-Pad97) -> /MCU/SP_4
- U31 pad 1: unconnected-(U31-Pad1) -> +5V
- U31 pad 8: unconnected-(U31-Pad8) -> +3V3
- U32 pad 1: unconnected-(U32-Pad1) -> +5V
- U32 pad 8: unconnected-(U32-Pad8) -> +3V3
- U33 pad 1: unconnected-(U33-Pad1) -> +5V
- U33 pad 8: unconnected-(U33-Pad8) -> +3V3
- U34 pad 1: unconnected-(U34-Pad1) -> +5V
- U34 pad 8: unconnected-(U34-Pad8) -> +3V3
- U35 pad 1: unconnected-(U35-Pad1) -> +3V3
- U35 pad 2: unconnected-(U35-Pad2) -> /Comms/USART_MCU_RX
- U35 pad 3: unconnected-(U35-Pad3) -> /Comms/USART_MCU_TX
- U35 pad 4: unconnected-(U35-Pad4) -> GND
- U35 pad 5: unconnected-(U35-Pad5) -> GND1
- U35 pad 6: unconnected-(U35-Pad6) -> /Comms/USART_UUT_RX
- U35 pad 7: unconnected-(U35-Pad7) -> /Comms/USART_UUT_TX
- U35 pad 8: unconnected-(U35-Pad8) -> +5V
- U36 pad 1: unconnected-(U36-Pad1) -> +3V3
- U36 pad 2: unconnected-(U36-Pad2) -> /Comms/CAN_RX
- U36 pad 3: unconnected-(U36-Pad3) -> /Comms/CAN_TX
- U36 pad 4: unconnected-(U36-Pad4) -> GND
- U36 pad 5: unconnected-(U36-Pad5) -> GND1
- U36 pad 6: unconnected-(U36-Pad6) -> /UUT_CAN_L
- U36 pad 7: unconnected-(U36-Pad7) -> /UUT_CAN_H
- U36 pad 8: unconnected-(U36-Pad8) -> +5V
- U37 pad 1: unconnected-(U37-Pad1) -> +3V3
- U37 pad 2: unconnected-(U37-Pad2) -> /Comms/I2C_SDA
- U37 pad 3: unconnected-(U37-Pad3) -> /Comms/I2C_SCL
- U37 pad 4: unconnected-(U37-Pad4) -> GND
- U37 pad 5: unconnected-(U37-Pad5) -> GND1
- U37 pad 6: unconnected-(U37-Pad6) -> /Comms/UUT_SCL
- U37 pad 7: unconnected-(U37-Pad7) -> /Comms/UUT_SDA
- U37 pad 8: unconnected-(U37-Pad8) -> +5V
- U38 pad 1: unconnected-(U38-Pad1) -> +3V3
- U38 pad 10: Net-(U38-Pad10) -> GND
- U38 pad 11: Net-(U38-Pad11) -> GND1
- U38 pad 16: unconnected-(U38-Pad16) -> /UUT_SPI_CIPO
- U38 pad 17: unconnected-(U38-Pad17) -> /UUT_SPI_COPI
- U38 pad 18: unconnected-(U38-Pad18) -> /UUT_SPI_SCK
- U38 pad 19: Net-(U38-Pad11) -> GND1
- U38 pad 2: Net-(U38-Pad10) -> GND
- U38 pad 20: unconnected-(U38-Pad20) -> +5V
- U38 pad 3: unconnected-(U38-Pad3) -> /Comms/SPI_SCK
- U38 pad 4: unconnected-(U38-Pad4) -> /Comms/SPI_COPI
- U38 pad 5: unconnected-(U38-Pad5) -> /Comms/SPI_CIPO
- U5 pad 1: unconnected-(U5-Pad1) -> +3V3
- U5 pad 2: +3V3 -> /MCU/PWM_1
- U5 pad 3: unconnected-(U5-Pad3) -> /MCU/PWM_2
- U5 pad 5: unconnected-(U5-Pad5) -> GND1
- U5 pad 6: Net-(U3-Pad43) -> /Timer IO/PWM_O_2
- U5 pad 7: unconnected-(U5-Pad7) -> /Timer IO/PWM_O_1
- U5 pad 8: unconnected-(U5-Pad8) -> +5V
- U6 pad 1: /Analogue Buffers/AI_S_4 -> /AI_S_4
- U6 pad 12: /Analogue Buffers/AI_S_3 -> /AI_S_3
- U6 pad 13: /Analogue Buffers/AI_S_0 -> /AI_S_0
- U6 pad 14: /Analogue Buffers/AI_S_1 -> /AI_S_1
- U6 pad 15: /Analogue Buffers/AI_S_2 -> /AI_S_2
- U6 pad 2: /Analogue Buffers/AI_S_6 -> /AI_S_6
- U6 pad 4: /Analogue Buffers/AI_S_7 -> /AI_S_7
- U6 pad 5: /Analogue Buffers/AI_S_5 -> /AI_S_5
- U7 pad 1: /Analogue Buffers/AI_S_12 -> /AI_S_12
- U7 pad 12: /Analogue Buffers/AI_S_11 -> /AI_S_11
- U7 pad 13: /Analogue Buffers/AI_S_8 -> /AI_S_8
- U7 pad 14: /Analogue Buffers/AI_S_9 -> /AI_S_9
- U7 pad 15: /Analogue Buffers/AI_S_10 -> /AI_S_10
- U7 pad 2: /Analogue Buffers/AI_S_14 -> /AI_S_14
- U7 pad 4: /Analogue Buffers/AI_S_15 -> /AI_S_15
- U7 pad 5: /Analogue Buffers/AI_S_13 -> /AI_S_13
- U8 pad 1: /Analogue Buffers/AI_F_4 -> /AI_F_4
- U8 pad 11: /Analogue Buffers/AI_F_3 -> /AI_F_3
- U8 pad 12: /Analogue Buffers/AI_F_0 -> /AI_F_0
- U8 pad 14: /Analogue Buffers/AI_F_1 -> /AI_F_1
- U8 pad 15: /Analogue Buffers/AI_F_2 -> /AI_F_2
- U8 pad 2: /Analogue Buffers/AI_F_6 -> /AI_F_6
- U8 pad 4: /Analogue Buffers/AI_F_7 -> /AI_F_7
- U8 pad 5: /Analogue Buffers/AI_F_5 -> /AI_F_5
Other:
- board outline added: 160 x 60 mm
